File: pcb-rpl-uph/usb-a.kicad_sch (KiCad schematic)
At the start: 7 parts, among them J2 USB3_A, U23 AP22811AW5-7, U5 USBLC6-2SC6

Commit message: Rename motherboard project, add models and footprints for M.2, USB-A, and USB-C
Parts:
- J3: renamed from J2; footprint nuc-12-carrier:USB3_A_CnC_Tech_1003-002-01100 -> local:USB3_A_CnC_Tech_1003-002-01100
- renumbered C51 to C17, C52 to C18, C44 to C19, D2 to D1, U23 to U1, U5 to U2

Commit message: refactor much of CPU schematic symbol
Other:
- note added: "TODO: common mode chokes overcurrent to CPU"
- note removed: "FLG to EC?"
Changed lines of the file:
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@@
     (effects (font (size 1.27 1.27)) (justify left bottom))
   )
-  (text "FLG to EC?" (at 113.03 60.96 0)
+  (text "TODO:\ncommon mode chokes\novercurrent to CPU" (at 106.68 130.81 0)
     (effects (font (size 1.27 1.27)) (justify left bottom))
   )

Commit message: USB PD input work in progress
Connections:
- net ~{FAULT}: now reaches U1.3 (FLG)
- net EN_VBUS: now reaches U1.4 (EN)
Other:
- note added: "TODO: common mode chokes"
- note removed: "EN from EC?"
- note removed: "TODO: common mode chokes overcurrent to CPU"
Changed lines of the file:
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@@
+    (stroke (width 0) (type default))
+  )
+  (wire (pts (xy 115.57 60.96) (xy 105.41 60.96))
     (stroke (width 0) (type default))
   )
@@
     (stroke (width 0) (type default))
   )
-  (text "EN from EC?" (at 74.93 58.42 0)
-    (effects (font (size 1.27 1.27)) (justify left bottom))
+  (wire (pts (xy 80.01 58.42) (xy 87.63 58.42))
+    (stroke (width 0) (type default))
   )
-  (text "TODO:\ncommon mode chokes\novercurrent to CPU" (at 106.68 130.81 0)
+  (text "TODO:\ncommon mode chokes" (at 106.68 130.81 0)
     (effects (font (size 1.27 1.27)) (justify left bottom))
   )
@@
     (effects (font (size 1.27 1.27)) (justify left bottom))
   )
+  (hierarchical_label "EN_VBUS" (shape input) (at 80.01 58.42 180) (fields_autoplaced)
+    (effects (font (size 1.27 1.27)) (justify right))
+  )
+  (hierarchical_label "~{FAULT}" (shape output) (at 115.57 60.96 0) (fields_autoplaced)
+    (effects (font (size 1.27 1.27)) (justify left))
+  )
   (hierarchical_label "USB{D+, D-, SSRX0+, SSRX0-, SSTX0+, SSTX0-}" (shape bidirectional) (at 64.77 71.12 180) (fields_autoplaced)
