File: pcb-rpl-uph/cpu_misc.kicad_sch (KiCad schematic)
At the start: 11 parts, among them U5 RPL_UPH_FCBGA1744

Commit message: add VCCINAUX
Parts:
- C33: footprint Capacitor_SMD:C_0402_1005Metric -> local:C_0402_1005Metric
Changed lines of the file:
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@@
       (effects (font (size 1.27 1.27)) (justify left))
     )
-    (property "Footprint" "Capacitor_SMD:C_0402_1005Metric" (at 410.5148 63.5 0)
+    (property "Footprint" "local:C_0402_1005Metric" (at 410.5148 63.5 0)
       (effects (font (size 1.27 1.27)) hide)
     )
