File: pcb-rpl-uph/vccinaux.kicad_sch (KiCad schematic)
At the start: 34 parts, among them Q14 CSD87355Q5D

Commit message: VCCCORE, VCCGT WIP
Parts:
- added C181 (x4): 10 uF, local:C_0805_2012Metric, symbol Device:C
- added C183: 47 uF, local:C_0603_1608Metric, symbol Device:C
- added R160: 100 k, local:R_0201_0603Metric, symbol Device:R
- added U5: RPL_UPH_FCBGA1744, local:RPL_UPH_FCBGA1744, symbol local:RPL_UPH_FCBGA1744
- L4: value 220 nH -> MHCC10040-R22M-R7; footprint Inductor_SMD:L_Bourns_SRR1210A -> Inductor_SMD:L_Chilisin_BMRG00101030
- R165, R166: value 10 -> 100
- U26: value ~ -> TPS51215ARUKR
- renumbered C184 to C187
Connections:
- net GND: now also C181.1, C181.1, C181.1, C181.1, C183.1
- net PGOOD: now also R160.2
- net VCCINAUX: now also U5.AL20 (VCCIN_AUX), U5.AL32 (VCCIN_AUX), U5.AN20 (VCCIN_AUX), U5.AN22 (VCCIN_AUX), U5.AN30 (VCCIN_AUX), U5.AN32 (VCCIN_AUX), U5.AN37 (VCCIN_AUX), U5.AP17 (VCCIN_AUX), U5.AP27 (VCCIN_AUX), U5.AP30 (VCCIN_AUX), U5.AP32 (VCCIN_AUX), U5.AP37 (VCCIN_AUX), U5.B3 (VCCIN_AUX), U5.D3 (VCCIN_AUX), U5.DH45 (VCCIN_AUX), U5.DJ41 (VCCIN_AUX), U5.DJ44 (VCCIN_AUX), U5.DK40 (VCCIN_AUX), U5.DK43 (VCCIN_AUX), U5.DK45 (VCCIN_AUX), U5.DL44 (VCCIN_AUX), U5.DM1 (VCCIN_AUX), U5.DM14 (VCCIN_AUX), U5.DM43 (VCCIN_AUX), U5.DP41 (VCCIN_AUX), U5.DP42 (VCCIN_AUX), U5.DR14 (VCCIN_AUX), U5.DR40 (VCCIN_AUX), U5.DT41 (VCCIN_AUX), U5.DU14 (VCCIN_AUX), U5.DU40 (VCCIN_AUX), U5.DV2 (VCCIN_AUX), U5.E1 (VCCIN_AUX), U5.ED2 (VCCIN_AUX), U5.EL2 (VCCIN_AUX), U5.F1 (VCCIN_AUX), U5.F3 (VCCIN_AUX), U5.G3 (VCCIN_AUX), U5.H4 (VCCIN_AUX), U5.J1 (VCCIN_AUX), U5.J3 (VCCIN_AUX), U5.L1 (VCCIN_AUX), U5.L3 (VCCIN_AUX), U5.N3 (VCCIN_AUX)
- net VCCINAUX_SENSE: now also U5.AF30 (VCCINAUX_SENSE)
- net VSSINAUX_SENSE: now also U5.AH30 (VSSINAUX_SENSE)
- net +VSW: now reaches Q14.1 (VIN)
- net +VSW: now also C181.2, C181.2, C181.2, C181.2
- new net VCCIN_AUX_FLTR: C183.2, U5.P1 (VCCIN_AUX_FLTR)
Other:
- note added: "TODO: proper inductor footprint"
- note added: "VCCIN_AUX 32 A max V00: 0 V V01: 1.1 V V10: 1.65 V V11: 1.8 V"
- note removed: "TODO: select inductor"
- note removed: "VCCIN_AUX 32 A max 480 uF minimum V00: 0 V V01: 1.1 V V10: 1.65 V V11: 1.8 V"
- moved on the sheet: C180, C181, C182, C183, C187, L4, Q14, R160, R161, R162, R163, R164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
