File: pcb-rpl-uph/vcc_core_gt.kicad_sch (KiCad schematic)
At the start: 36 parts, among them U27 RT3624, U5 RPL_UPH_FCBGA1744

Commit message: core power work in progress
Parts:
- removed U28: ~, Package_DFN_QFN:DFN-8-1EP_2x2mm_P0.5mm_EP0.6x1.2mm, symbol local:RT9610C
- added C183: 4.7 uF, local:C_0603_1608Metric, symbol Device:C
- added C183: 470 nF, local:C_0603_1608Metric, symbol Device:C
- added C183: 220 nF, local:C_0402_1005Metric, symbol Device:C
- added R168: 10 k, local:R_0201_0603Metric, symbol Device:R
- added R169: 2.2, local:R_0603_1608Metric, symbol Device:R
- added R176, R177, R178, R193, R194, R195, R196, R197, R198, R199, R200, R201, R203: TBD, local:R_0201_0603Metric, symbol Device:R
- added R202: 3.9, local:R_0402_1005Metric, symbol Device:R
- added TH1, TH2, TH3, TH4: 100k B4250, local:R_0402_1005Metric, symbol Device:Thermistor
Connections:
- net +5V: now also R169.2; no longer U27.50 (VCC)
- net GND: now also C183.1, C183.1, C183.1, R177.1, R194.1, R197.1, R200.1
- net PC3/ISEN+: now reaches U27.1 (ISEN3P)
- net VREF_SPS: now reaches U27.13 (VREF_SPS)
- net VREF_SPS: now also C183.2
- net VR_READY: now reaches U27.14 (VR_READY)
- net VCLK: now reaches U27.15 (VCLK)
- net VDIO: now reaches U27.16 (VDIO)
- net ~{ALERT}: now reaches U27.17 (~{ALERT})
- net ~{VR_HOT}: now reaches U27.18 (~{VR_HOT})
- net IMON: now reaches U27.19 (IMON)
- net IMON: now also R199.2, TH4.2
- net PC3/ISEN-: now reaches U27.2 (ISEN3N)
- net VREF: now reaches U27.20 (VREF)
- net VREF: now also R178.2, R195.2, R198.2, R201.2, R202.2, R203.1
- net IMONA: now reaches U27.21 (IMONA)
- net IMONA: now also R196.2, TH3.2
- net TSEN: now reaches U27.22 (TSEN)
- net TSEN: now also R176.2, TH1.2
- net TSENA: now reaches U27.23 (TSENA)
- net TSENA: now also R193.2, TH2.2
- net IMON_AUX: now reaches U27.28 (IMON_AUX)
- net IMON_AUX: now also R203.2
- net at U27.3 (ISEN4N): now also U27.4 (ISEN4P), R168.1
- net PG2/ISEN+: now reaches U27.34 (ISENA2N)
- net PG2/ISEN-: now reaches U27.35 (ISENA2P)
- net PG1/ISEN+: now reaches U27.36 (ISENA1P)
- net PG1/ISEN-: now reaches U27.37 (ISENA1N)
- net PG2/PWM: now reaches U27.43 (PWMA2)
- net PG1/PWM: now reaches U27.44 (PWMA1)
- net PC1/PWM: now reaches U27.45 (PWM1)
- net PC2/PWM: now reaches U27.46 (PWM2)
- net PC3/PWM: now reaches U27.48 (PWM3)
- net PC2/ISEN+: now reaches U27.5 (ISEN2P)
- net VRON: now reaches U27.51 (VRON)
- net PC2/ISEN-: now reaches U27.6 (ISEN2N)
- net PC1/ISEN-: now reaches U27.7 (ISEN1N)
- net PC1/ISEN+: now reaches U27.8 (ISEN1P)
- new net: C183.2, R202.1
- new net IMON1: R199.1, R200.2, R201.1, TH4.1
- new net IMONA1: R196.1, R197.2, R198.1, TH3.1
- new net TSEN1: R176.1, R177.2, R178.1, TH1.1
- new net TSENA1: R193.1, R194.2, R195.1, TH2.1
- new net VCC: C183.2, R168.2, R169.1, U27.50 (VCC)
- no-connect marks 0 -> 1
Other:
- added sheet PC1 (phase.kicad_sch)
- added sheet PC2 (phase.kicad_sch)
- added sheet PC3 (phase.kicad_sch)
- added sheet PG1 (phase.kicad_sch)
- added sheet PG2 (phase.kicad_sch)
- note added: "1.3 V nominal"
- note added: "Place IMON thermistors near inductor of associated phase 1"
- note added: "Place thermistors near hottest part of voltage regulator TSENA is GT, TSEN is core"
- moved on the sheet: C183, C187, U27
